Commit message: feat: robot description, gazebo elements, and dynamic attachment feasible by encapsulating in xacro

File: src/mycobot_320/urdf/320_urdf/mycobot_320.xacro (robot description, xacro)
@@ -8,6 +8,6 @@
     <inertial>
       <origin xyz="-0.00314201374155656 -0.000316576969441296 0.0310618347596631" rpy="0 0 0" />
-      <mass value="0.126527076069415" />
-      <inertia ixx="0.000112288059520224" ixy="-9.28284765851997E-07" ixz="1.66442838582405E-07" iyy="0.000108773547634347" iyz="-5.48664083571427E-07" izz="0.000142112834287267" />
+      <mass value="0.92353" />
+      <inertia ixx="0.00084401" ixy="-7.3631E-06" ixz="1.4091E-06" iyy="0.00083129" iyz="-4.0382E-06" izz="0.0010931" />
     </inertial>
     <visual>
@@ -30,6 +30,6 @@
     <inertial>
       <origin xyz="-4.65008859791595E-06 -0.00713845775566615 0.039058845834672" rpy="0 0 0" />
-      <mass value="0.0427054445276861" />
-      <inertia ixx="3.72257027289962E-05" ixy="6.57695397778541E-09" ixz="-2.01754415740566E-08" iyy="3.78334224688226E-05" iyz="1.08516622017588E-05" izz="1.74950666609677E-05" />
+      <mass value="0.3331" />
+      <inertia ixx="0.00029036" ixy="5.13E-08" ixz="-1.5737E-07" iyy="0.0002951" iyz="8.4643E-05" izz="0.00013646" />
     </inertial>
     <visual>
@@ -59,6 +59,6 @@
     <inertial>
       <origin xyz="-0.0513897959483668 1.03416109062133E-07 0.0428557705148588" rpy="0 0 0" />
-      <mass value="0.0376782548805202" />
-      <inertia ixx="1.11164690983472E-05" ixy="-6.38474472311225E-09" ixz="-2.0084433833182E-06" iyy="9.00231742503222E-05" iyz="3.96245537473233E-09" izz="9.52053931799855E-05" />
+      <mass value="0.29389" />
+      <inertia ixx="8.6708E-05" ixy="-4.9801E-08" ixz="-1.5666E-05" iyy="0.00070218" iyz="3.0907E-08" izz="0.0007426" />
     </inertial>
     <visual>
@@ -88,6 +88,6 @@
     <inertial>
       <origin xyz="-0.0437220859914132 -1.2774481847333E-06 0.00135653065468257" rpy="0 0 0" />
-      <mass value="0.0533399040690726" />
-      <inertia ixx="1.3694550753436E-05" ixy="-4.86029624235192E-09" ixz="-4.04939679872146E-06" iyy="9.74114113250282E-05" iyz="-2.54559379960044E-09" izz="0.000101615718356252" />
+      <mass value="0.41605" />
+      <inertia ixx="0.00010682" ixy="-3.791E-08" ixz="-3.1585E-05" iyy="0.00075981" iyz="-1.9856E-08" izz="0.0007926" />
     </inertial>
     <visual>
@@ -117,6 +117,6 @@
     <inertial>
       <origin xyz="-1.40520224535812E-05 -0.0076816570577589 0.0230103540086662" rpy="0 0 0" />
-      <mass value="0.0240733217897794" />
-      <inertia ixx="9.33009576664887E-06" ixy="-1.25594881163816E-10" ixz="2.4324214522356E-09" iyy="7.82113831853559E-06" iyz="3.31133798836023E-06" izz="7.74288688073051E-06" />
+      <mass value="0.18777" />
+      <inertia ixx="7.2775E-05" ixy="-9.7964E-10" ixz="1.8973E-08" iyy="6.1005E-05" iyz="2.5828E-05" izz="6.0395E-05" />
     </inertial>
     <visual>
@@ -146,6 +146,6 @@
     <inertial>
       <origin xyz="0.000112529211153511 0.00287540778498707 0.0396485032237697" rpy="0 0 0" />
-      <mass value="0.0288700851686918" />
-      <inertia ixx="1.31118730631263E-05" ixy="-2.83589105523716E-08" ixz="-1.1232400033724E-08" iyy="1.30202251952408E-05" iyz="-2.99882844237461E-06" izz="8.33442454575535E-06" />
+      <mass value="0.22519" />
+      <inertia ixx="0.00010227" ixy="-2.212E-07" ixz="-8.7613E-08" iyy="0.00010156" iyz="-2.3391E-05" izz="6.5009E-05" />
     </inertial>
     <visual>
@@ -175,6 +175,6 @@
     <inertial>
       <origin xyz="-1.18357394707225E-06 -3.05824490363232E-06 0.0305489098542017" rpy="0 0 0" />
-      <mass value="0.00770532070308737" />
-      <inertia ixx="8.40243449154729E-07" ixy="7.46728835461358E-14" ixz="5.37605897551446E-11" iyy="8.40609096397143E-07" iyz="-1.3115260747023E-10" izz="1.35522228863536E-06" />
+      <mass value="0.060102" />
+      <inertia ixx="6.5539E-06" ixy="5.8245E-13" ixz="4.1933E-10" iyy="6.5568E-06" iyz="-1.023E-09" izz="1.0571E-05" />
     </inertial>
     <visual>

File: src/mycobot_320/urdf/mycobot_robot_macro.xacro (robot description, xacro)
@@ -1,11 +1,12 @@
 <?xml version="1.0" encoding='utf-8'?>
-<robot xmlns:xacro="http://ros.org/wiki/xacro" name="mycobot_pro_robot" >
-  <xacro:macro name="mycobot_pro_robot_macro" params="prefix:='' namespace:='xarm' limited:='false' effort_control:='false'
-    velocity_control:='false' attach_to:='world' xyz:='0 0 0' rpy:='0 0 0' load_gazebo_plugin:='true' ">
+<robot xmlns:xacro="http://ros.org/wiki/xacro">
+  <xacro:macro name="mycobot_pro_robot_macro" params="prefix:='' namespace:='xarm' limited:='false' effort_control:='false' velocity_control:='false' attach_to:='world' xyz:='0 0 0' rpy:='0 0 0' load_gazebo_plugin:='true' camera_sensor='true' ">
     <!-- include mycobot relative macros: -->
-    <xacro:include filename="$(find mycobot_320)/urdf/320_urdf/mycobot_320.xacro" />
+    <xacro:include filename="$(find mycobot_320)/urdf/320_urdf/mycobot_320.urdf" />
+    <!-- include gazebo elements -->
+    <xacro:include filename="$(find mycobot_320)/urdf/mycobot_robot.gazebo.xacro"/>
     <!-- add one world link if no 'attach_to' specified  -->
     <xacro:if value="${attach_to == 'world'}">
-      <link name="world" />
+      <link name="world"/>
     </xacro:if>
     <joint name="world_joint" type="fixed">
@@ -14,4 +15,8 @@
       <origin xyz="${xyz}" rpy="${rpy}" />
     </joint>
+    <!-- include the camera sensor mounted on the robotic arm if sensor is true -->
+    <xacro:if value="${camera_sensor == 'true'}">
+      <xacro:include filename="$(find mycobot_320)/urdf/mycobot_robot.sensor.xacro" />
+    </xacro:if>
   </xacro:macro>
 </robot>
