Commit message: fix: xacro boolean parameter issue resolved

File: src/mycobot_320/urdf/mycobot_robot.urdf.xacro (robot description, xacro)
@@ -3,6 +3,7 @@
   <xacro:arg name="ros_namespace" default="mycobot_pro"/>
   <xacro:arg name="attach_to" default="world"/>
+  <xacro:arg name="camera_sensor" default="True"/>
   <!-- load mycobot_pro robot -->
   <xacro:include filename="$(find mycobot_320)/urdf/mycobot_robot_macro.xacro" />
-  <xacro:mycobot_pro_robot_macro attach_to="$(arg attach_to)"/>
+  <xacro:mycobot_pro_robot_macro camera_sensor="$(arg camera_sensor)" attach_to="$(arg attach_to)"/>
 </robot>

File: src/mycobot_320/urdf/mycobot_robot_macro.xacro (robot description, xacro)
@@ -1,5 +1,5 @@
 <?xml version="1.0" encoding='utf-8'?>
 <robot xmlns:xacro="http://ros.org/wiki/xacro">
-  <xacro:macro name="mycobot_pro_robot_macro" params="prefix:='' namespace:='xarm' limited:='false' effort_control:='false' velocity_control:='false' attach_to:='world' xyz:='0 0 0' rpy:='0 0 0' load_gazebo_plugin:='true' camera_sensor='true' ">
+  <xacro:macro name="mycobot_pro_robot_macro" params="prefix:='' attach_to:='world' xyz:='0 0 0' rpy:='0 0 0' camera_sensor:=False ">
     <!-- include mycobot relative macros: -->
     <xacro:include filename="$(find mycobot_320)/urdf/320_urdf/mycobot_320.urdf" />
@@ -16,5 +16,5 @@
     </joint>
     <!-- include the camera sensor mounted on the robotic arm if sensor is true -->
-    <xacro:if value="${camera_sensor == 'true'}">
+    <xacro:if value="${camera_sensor == True}">
       <xacro:include filename="$(find mycobot_320)/urdf/mycobot_robot.sensor.xacro" />
     </xacro:if>
