Commit message: enhancement: fixed toilet urdf to world with rigit joint

File: src/toilet_urdf/urdf/toilet_urdf.xacro (robot description, xacro)
@@ -6,6 +6,17 @@
   xmlns:xacro="http://ros.org/wiki/xacro"
   name="toilet_urdf">
+  <link name="world"/>
+  <link name="toilet_virtual"/>
+  <joint name="toilet_virtual_joint" type="fixed">
+    <parent link="toilet_virtual"/>
+    <child link="toilet_base"/>
+  </joint>
+  <joint name="world_joint" type="fixed">
+    <origin xyz="0.5 -0.5 -0.2" rpy="0 0 -1.51"/>
+    <parent link="world"/>
+    <child link="toilet_virtual"/>
+  </joint>
   <link
-    name="base_link">
+    name="toilet_base">
     <inertial>
       <origin
@@ -93,5 +104,5 @@
       rpy="1.5708 0 0" />
     <parent
-      link="base_link" />
+      link="toilet_base" />
     <child
       link="toilet_shaft_link" />
