Commit message: enhancement: converted hivebot_trolley from urdf to xacro file

File: src/hivebot_trolley/urdf/hivebot_trolley.xacro (robot description, xacro)
@@ -4,5 +4,5 @@
      For more information, please see http://wiki.ros.org/sw_urdf_exporter -->
 <robot
-  name="hivebot_trolley">
+  name="hivebot_trolley" xmlns:xacro="http://www.ros.org/wiki/xacro">
   <link
     name="base_link">
@@ -12,12 +12,12 @@
         rpy="0 0 0" />
       <mass
-        value="23.4644604067189" />
-      <inertia
-        ixx="0.443716606385079"
-        ixy="1.51028178972321E-16"
-        ixz="0.00342987078268199"
-        iyy="0.784701467555992"
-        iyz="9.75264500412178E-19"
-        izz="1.20292332901758" />
+        value="63.354" />
+      <inertia
+        ixx="1.198"
+        ixy="3.8905E-16"
+        ixz="0.0092607"
+        iyy="2.1187"
+        iyz="2.6213E-18"
+        izz="3.2479" />
     </inertial>
     <visual>
@@ -32,5 +32,5 @@
         name="">
         <color
-          rgba="0.792156862745098 0.819607843137255 0.933333333333333 1" />
+          rgba="0.89804 0.91765 0.92941 1" />
       </material>
     </visual>
@@ -52,12 +52,12 @@
         rpy="0 0 0" />
       <mass
-        value="0.0327823001646924" />
-      <inertia
-        ixx="1.83921920866059E-05"
-        ixy="3.24615009351937E-21"
-        ixz="-1.54550847789467E-22"
-        iyy="1.83921920866059E-05"
-        iyz="1.24661932029889E-23"
-        izz="3.66220350741116E-05" />
+        value="0.088512" />
+      <inertia
+        ixx="4.9659E-05"
+        ixy="8.7646E-21"
+        ixz="-4.1729E-22"
+        iyy="4.9659E-05"
+        iyz="3.3659E-23"
+        izz="9.8879E-05" />
     </inertial>
     <visual>
@@ -72,5 +72,5 @@
         name="">
         <color
-          rgba="0.792156862745098 0.819607843137255 0.933333333333333 1" />
+          rgba="0.89804 0.91765 0.92941 1" />
       </material>
     </visual>
@@ -105,12 +105,12 @@
         rpy="0 0 0" />
       <mass
-        value="0.150983674432007" />
-      <inertia
-        ixx="0.00028266058025081"
-        ixy="-3.21116342948743E-20"
-        ixz="2.79944389067546E-19"
-        iyy="0.000195595027956607"
-        iyz="9.17390835065707E-20"
-        izz="0.000185655183273928" />
+        value="0.40766" />
+      <inertia
+        ixx="0.00076318"
+        ixy="-8.8118E-20"
+        ixz="7.5894E-19"
+        iyy="0.00052811"
+        iyz="2.369E-19"
+        izz="0.00050127" />
     </inertial>
     <visual>
@@ -125,5 +125,5 @@
         name="">
         <color
-          rgba="0.792156862745098 0.819607843137255 0.933333333333333 1" />
+          rgba="0.89804 0.91765 0.92941 1" />
       </material>
     </visual>
@@ -158,12 +158,12 @@
         rpy="0 0 0" />
       <mass
-        value="0.642809126832642" />
-      <inertia
-        ixx="0.000780813338623139"
-        ixy="5.42101086242752E-20"
-        ixz="-6.55230197504303E-20"
-        iyy="0.00078081333862314"
-        iyz="-1.84261108894285E-19"
-        izz="0.00127745325926734" />
+        value="1.7356" />
+      <inertia
+        ixx="0.0021082"
+        ixy="3.2526E-19"
+        ixz="-1.6963E-19"
+        iyy="0.0021082"
+        iyz="-4.6684E-19"
+        izz="0.0034491" />
     </inertial>
     <visual>
@@ -211,12 +211,12 @@
         rpy="0 0 0" />
       <mass
-        value="0.0327823001646925" />
-      <inertia
-        ixx="1.83921920866059E-05"
-        ixy="4.93527744713229E-21"
-        ixz="-5.06886009705894E-23"
-        iyy="1.83921920866059E-05"
-        iyz="-2.42774695441036E-22"
-        izz="3.66220350741116E-05" />
+        value="0.088512" />
+      <inertia
+        ixx="4.9659E-05"
+        ixy="1.3325E-20"
+        ixz="-1.3686E-22"
+        iyy="4.9659E-05"
+        iyz="-6.5549E-22"
+        izz="9.8879E-05" />
     </inertial>
     <visual>
@@ -264,12 +264,12 @@
         rpy="0 0 0" />
       <mass
-        value="0.150983674432007" />
-      <inertia
-        ixx="0.00028266058025081"
-        ixy="2.48099744005913E-20"
-        ixz="-5.8699383244723E-19"
-        iyy="0.000195595027956607"
-        iyz="8.44021330596004E-20"
-        izz="0.000185655183273928" />
+        value="0.40766" />
+      <inertia
+        ixx="0.00076318"
+        ixy="6.7699E-20"
+        ixz="-1.589E-18"
+        iyy="0.00052811"
+        iyz="2.4104E-19"
+        izz="0.00050127" />
     </inertial>
     <visual>
@@ -317,12 +317,12 @@
         rpy="0 0 0" />
       <mass
-        value="0.642809126832642" />
-      <inertia
-        ixx="0.000780813338623139"
-        ixy="-5.42101086242752E-20"
-        ixz="4.90097043911794E-19"
-        iyy="0.000780813338623139"
-        iyz="-4.72387687152462E-19"
-        izz="0.00127745325926734" />
+        value="1.7356" />
+      <inertia
+        ixx="0.0021082"
+        ixy="-3.2526E-19"
+        ixz="1.2945E-18"
+        iyy="0.0021082"
+        iyz="-1.3425E-18"
+        izz="0.0034491" />
     </inertial>
     <visual>
@@ -370,12 +370,12 @@
         rpy="0 0 0" />
       <mass
-        value="1.36689710972196" />
-      <inertia
-        ixx="0.00338021767437179"
-        ixy="2.06305140072641E-19"
-        ixz="-2.77319256608588E-19"
-        iyy="0.00382021767437179"
-        iyz="-1.2413112864934E-19"
-        izz="0.00249215534678811" />
+        value="3.6906" />
+      <inertia
+        ixx="0.0091266"
+        ixy="5.5702E-19"
+        ixz="-7.4876E-19"
+        iyy="0.010315"
+        iyz="-3.3515E-19"
+        izz="0.0067288" />
     </inertial>
     <visual>
@@ -423,12 +423,12 @@
         rpy="0 0 0" />
       <mass
-        value="2.69353870933482" />
-      <inertia
-        ixx="0.00949511675813368"
-        ixy="5.29395592033938E-23"
-        ixz="9.95024472665243E-19"
-        iyy="0.00949511675813367"
-        iyz="-1.1541177720628E-18"
-        izz="0.0161171255596435" />
+        value="7.2726" />
+      <inertia
+        ixx="0.025637"
+        ixy="2.647E-22"
+        ixz="2.6866E-18"
+        iyy="0.025637"
+        iyz="-3.1161E-18"
+        izz="0.043516" />
     </inertial>
     <visual>
@@ -476,12 +476,12 @@
         rpy="0 0 0" />
       <mass
-        value="1.36689710972196" />
-      <inertia
-        ixx="0.00338021767437178"
-        ixy="3.21237840152391E-19"
-        ixz="-1.88824243478581E-19"
-        iyy="0.00382021767437178"
-        iyz="-1.63935584020256E-21"
-        izz="0.00249215534678811" />
+        value="3.6906" />
+      <inertia
+        ixx="0.0091266"
+        ixy="8.6734E-19"
+        ixz="-5.0983E-19"
+        iyy="0.010315"
+        iyz="2.5555E-20"
+        izz="0.0067288" />
     </inertial>
     <visual>
@@ -529,12 +529,12 @@
         rpy="0 0 0" />
       <mass
-        value="2.69353870933482" />
-      <inertia
-        ixx="0.00949511675813368"
+        value="7.2726" />
+      <inertia
+        ixx="0.025637"
         ixy="0"
-        ixz="1.26731753157619E-18"
-        iyy="0.00949511675813368"
-        iyz="-1.52133972476596E-18"
-        izz="0.0161171255596436" />
+        ixz="3.4218E-18"
+        iyy="0.025637"
+        iyz="-4.1076E-18"
+        izz="0.043516" />
     </inertial>
     <visual>
@@ -582,12 +582,12 @@
         rpy="0 0 0" />
       <mass
-        value="5.75784" />
-      <inertia
-        ixx="0.369158792655726"
-        ixy="2.49402192883461E-18"
-        ixz="5.73478237026073E-17"
-        iyy="0.387658995375726"
-        iyz="3.63659399409593E-17"
-        izz="0.02826234816" />
+        value="15.546" />
+      <inertia
+        ixx="0.99673"
+        ixy="6.6037E-18"
+        ixz="1.5535E-16"
+        iyy="1.0467"
+        iyz="9.6464E-17"
+        izz="0.076308" />
     </inertial>
     <visual>
@@ -635,12 +635,12 @@
         rpy="0 0 0" />
       <mass
-        value="1.43838725877128" />
-      <inertia
-        ixx="0.00345361373947357"
-        ixy="1.45609786108984E-19"
-        ixz="-1.2659665150112E-19"
-        iyy="0.00290597229871286"
-        iyz="-6.51769155242515E-19"
-        izz="0.00290766425871286" />
+        value="3.8836" />
+      <inertia
+        ixx="0.0093248"
+        ixy="4.3129E-19"
+        ixz="1.0113E-20"
+        iyy="0.0078461"
+        iyz="-1.9951E-18"
+        izz="0.0078507" />
     </inertial>
     <visual>
@@ -693,12 +693,12 @@
         rpy="0 0 0" />
       <mass
-        value="39.1078118021391" />
-      <inertia
-        ixx="1.55288148334587"
-        ixy="-0.00153801040030465"
-        ixz="0.00220493109382033"
-        iyy="1.67301946819098"
-        iyz="0.0166316312278493"
-        izz="1.1231420016058" />
+        value="82.748" />
+      <inertia
+        ixx="3.3922"
+        ixy="-0.0022233"
+        ixz="0.002369"
+        iyy="3.782"
+        iyz="0.020109"
+        izz="1.8643" />
     </inertial>
     <visual>
@@ -713,5 +713,5 @@
         name="">
         <color
-          rgba="0.792156862745098 0.819607843137255 0.933333333333333 1" />
+          rgba="0.89804 0.91765 0.92941 1" />
       </material>
     </visual>
@@ -746,12 +746,12 @@
         rpy="0 0 0" />
       <mass
-        value="1.71577433388231" />
-      <inertia
-        ixx="0.0128235955145912"
-        ixy="-7.18271089932621E-06"
-        ixz="1.93339625511969E-05"
-        iyy="0.0117484833677518"
-        iyz="1.88568302746812E-06"
-        izz="0.0244481959322745" />
+        value="2.0589" />
+      <inertia
+        ixx="0.015388"
+        ixy="-8.6193E-06"
+        ixz="2.3201E-05"
+        iyy="0.014098"
+        iyz="2.2628E-06"
+        izz="0.029338" />
     </inertial>
     <visual>
@@ -766,5 +766,5 @@
         name="">
         <color
-          rgba="0.792156862745098 0.819607843137255 0.933333333333333 1" />
+          rgba="1 1 1 0.3" />
       </material>
     </visual>
@@ -799,12 +799,12 @@
         rpy="0 0 0" />
       <mass
-        value="0.113687986940389" />
-      <inertia
-        ixx="0.000111445471191984"
-        ixy="-6.15789915572864E-11"
-        ixz="2.32192465433345E-08"
-        iyy="0.000413028900787828"
-        iyz="2.72645884829236E-08"
-        izz="0.000302229544189519" />
+        value="0.886766298135032" />
+      <inertia
+        ixx="0.000869274675297478"
+        ixy="-4.8031613415315E-10"
+        ixz="1.8111012303801E-07"
+        iyy="0.00322162542614506"
+        iyz="2.12663790167015E-07"
+        izz="0.00235739044467824" />
     </inertial>
     <visual>
@@ -819,5 +819,5 @@
         name="">
         <color
-          rgba="0.792156862745098 0.819607843137255 0.933333333333333 1" />
+          rgba="0.529411764705882 0.549019607843137 0.549019607843137 1" />
       </material>
     </visual>
@@ -852,12 +852,12 @@
         rpy="0 0 0" />
       <mass
-        value="0.383705226392601" />
-      <inertia
-        ixx="0.000225586911534695"
-        ixy="2.06897283647009E-19"
-        ixz="1.39338231937946E-18"
-        iyy="0.00803378140369941"
-        iyz="1.95575888623689E-20"
-        izz="0.00785136133013388" />
+        value="1.03600411126002" />
+      <inertia
+        ixx="0.000609084661143678"
+        ixy="5.58622665846924E-19"
+        ixz="3.76213226232454E-18"
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
Commit message: fix: hivebot_trolley coordinates and spawn in gazebo

File: src/hivebot_trolley/urdf/hivebot_trolley.xacro (robot description, xacro)
@@ -3,21 +3,26 @@
      Commit Version: 1.6.0-1-g15f4949  Build Version: 1.6.7594.29634
      For more information, please see http://wiki.ros.org/sw_urdf_exporter -->
-<robot
-  name="hivebot_trolley" xmlns:xacro="http://www.ros.org/wiki/xacro">
+<robot name="hivebot_trolley">
+  <link name="base_footprint" xmlns:xacro="http://www.ros.org/wiki/xacro"/>
+  <joint name="base_joint" type="fixed">
+    <origin xyz="0 0 0.05" rpy="0 0 0" />
+    <parent link="base_footprint"/>
+    <child link="base_link" />
+  </joint>
   <link
     name="base_link">
     <inertial>
       <origin
-        xyz="0.0235732763735559 -1.16301105845676E-16 -0.0393476182287232"
-        rpy="0 0 0" />
-      <mass
-        value="63.354" />
-      <inertia
-        ixx="1.198"
-        ixy="3.8905E-16"
-        ixz="0.0092607"
-        iyy="2.1187"
-        iyz="2.6213E-18"
-        izz="3.2479" />
+        xyz="0.0235732763735559 -1.16156711654192E-16 -0.0393476182287232"
+        rpy="0 0 0" />
+      <mass
+        value="63.3540430981409" />
+      <inertia
+        ixx="1.19803483723971"
+        ixy="3.94354928014663E-16"
+        ixz="0.00926065111324139"
+        iyy="2.11869396240118"
+        iyz="2.70482966665085E-18"
+        izz="3.24789298834746" />
     </inertial>
     <visual>
@@ -32,5 +37,5 @@
         name="">
         <color
-          rgba="0.89804 0.91765 0.92941 1" />
+          rgba="0.898039215686275 0.917647058823529 0.929411764705882 1" />
       </material>
     </visual>
@@ -45,19 +50,32 @@
     </collision>
   </link>
+  <joint
+    name="compartment-2-to-base"
+    type="fixed">
+    <origin
+      xyz="-0.2 -0.125 0"
+      rpy="0 0 0" />
+    <parent
+      link="base_link" />
+    <child
+      link="compartment-2" />
+    <axis
+      xyz="0 0 0" />
+  </joint>
   <link
     name="front_wheel_mount_plate_1">
     <inertial>
       <origin
-        xyz="0 0 0.00372376098180308"
-        rpy="0 0 0" />
-      <mass
-        value="0.088512" />
-      <inertia
-        ixx="4.9659E-05"
-        ixy="8.7646E-21"
-        ixz="-4.1729E-22"
-        iyy="4.9659E-05"
-        iyz="3.3659E-23"
-        izz="9.8879E-05" />
+        xyz="0 0 0.00372376098180309"
+        rpy="0 0 0" />
+      <mass
+        value="0.0885122104446696" />
+      <inertia
+        ixx="4.96589186338358E-05"
+        ixy="8.76460525250229E-21"
+        ixz="4.57370748529084E-22"
+        iyy="4.96589186338358E-05"
+        iyz="-1.38813531491213E-23"
+        izz="9.88794947001013E-05" />
     </inertial>
     <visual>
@@ -72,5 +90,5 @@
         name="">
         <color
-          rgba="0.89804 0.91765 0.92941 1" />
+          rgba="0.898039215686275 0.917647058823529 0.929411764705882 1" />
       </material>
     </visual>
@@ -90,5 +108,5 @@
     <origin
       xyz="0.28 -0.205 -0.086"
-      rpy="0 0 3.1416" />
+      rpy="0 0 0" />
     <parent
       link="base_link" />
@@ -102,15 +120,15 @@
     <inertial>
       <origin
-        xyz="0 0.0353498305391302 5.55111512312578E-17"
-        rpy="0 0 0" />
-      <mass
-        value="0.40766" />
-      <inertia
-        ixx="0.00076318"
-        ixy="-8.8118E-20"
-        ixz="7.5894E-19"
-        iyy="0.00052811"
-        iyz="2.369E-19"
-        izz="0.00050127" />
+        xyz="0 -5.55111512312578E-17 -0.0353498305391301"
+        rpy="0 0 0" />
+      <mass
+        value="0.40765592096642" />
+      <inertia
+        ixx="0.000762776791330026"
+        ixy="1.03138220220553E-05"
+        ixz="6.91311896835273E-20"
+        iyy="0.000501675770186767"
+        iyz="-1.75192826322455E-19"
+        izz="0.000528106575482838" />
     </inertial>
     <visual>
@@ -125,5 +143,5 @@
         name="">
         <color
-          rgba="0.89804 0.91765 0.92941 1" />
+          rgba="0.898039215686275 0.917647058823529 0.929411764705882 1" />
       </material>
     </visual>
@@ -143,5 +161,5 @@
     <origin
       xyz="0 0 0"
-      rpy="-1.5708 0 -3.1022" />
+      rpy="0 0 0" />
     <parent
       link="front_wheel_mount_plate_1" />
@@ -149,5 +167,5 @@
       link="front_wheel_holder_1" />
     <axis
-      xyz="0 1 0" />
+      xyz="0 0 -1" />
   </joint>
   <link
@@ -155,15 +173,15 @@
     <inertial>
       <origin
-        xyz="0 0 5.55111512312578E-17"
-        rpy="0 0 0" />
-      <mass
-        value="1.7356" />
-      <inertia
-        ixx="0.0021082"
-        ixy="3.2526E-19"
-        ixz="-1.6963E-19"
-        iyy="0.0021082"
-        iyz="-4.6684E-19"
-        izz="0.0034491" />
+        xyz="5.55111512312578E-17 8.32667268468867E-17 -5.55111512312578E-17"
+        rpy="0 0 0" />
+      <mass
+        value="1.73558464244813" />
+      <inertia
+        ixx="0.00211027858785498"
+        ixy="-5.2803822366633E-05"
+        ixz="1.94419187005969E-19"
+        iyy="0.00344704122644933"
+        iyz="-2.97963645002492E-19"
+        izz="0.00210819601428248" />
     </inertial>
     <visual>
@@ -178,5 +196,5 @@
         name="">
         <color
-          rgba="0.792156862745098 0.819607843137255 0.933333333333333 1" />
+          rgba="0.898039215686275 0.917647058823529 0.929411764705882 1" />
       </material>
     </visual>
@@ -195,6 +213,6 @@
     type="continuous">
     <origin
-      xyz="0 0.081 0"
-      rpy="0 0 1.9085" />
+      xyz="0 0 -0.081"
+      rpy="0 0 0" />
     <parent
       link="front_wheel_holder_1" />
@@ -202,5 +220,5 @@
       link="front_wheel_1" />
     <axis
-      xyz="0 0 1" />
+      xyz="-0.0394091875345171 0.99922315622581 0" />
   </joint>
   <link
@@ -208,15 +226,15 @@
     <inertial>
       <origin
-        xyz="0 -2.77555756156289E-17 0.00372376098180308"
-        rpy="0 0 0" />
-      <mass
-        value="0.088512" />
-      <inertia
-        ixx="4.9659E-05"
-        ixy="1.3325E-20"
-        ixz="-1.3686E-22"
-        iyy="4.9659E-05"
-        iyz="-6.5549E-22"
-        izz="9.8879E-05" />
+        xyz="0 -2.77555756156289E-17 0.00372376098180309"
+        rpy="0 0 0" />
+      <mass
+        value="0.0885122104446697" />
+      <inertia
+        ixx="4.96589186338359E-05"
+        ixy="1.33252491072572E-20"
+        ixz="1.0447510163914E-22"
+        iyy="4.96589186338359E-05"
+        iyz="6.3556804032152E-22"
+        izz="9.88794947001014E-05" />
     </inertial>
     <visual>
@@ -231,5 +249,5 @@
         name="">
         <color
-          rgba="0.792156862745098 0.819607843137255 0.933333333333333 1" />
+          rgba="0.898039215686275 0.917647058823529 0.929411764705882 1" />
       </material>
     </visual>
@@ -249,5 +267,5 @@
     <origin
       xyz="0.28 0.205 -0.086"
-      rpy="0 0 3.1416" />
+      rpy="0 0 0" />
     <parent
       link="base_link" />
@@ -261,15 +279,15 @@
     <inertial>
       <origin
-        xyz="0 0.0353498305391302 -1.38777878078145E-16"
-        rpy="0 0 0" />
-      <mass
-        value="0.40766" />
-      <inertia
-        ixx="0.00076318"
-        ixy="6.7699E-20"
-        ixz="-1.589E-18"
-        iyy="0.00052811"
-        iyz="2.4104E-19"
-        izz="0.00050127" />
+        xyz="-5.55111512312578E-17 -5.55111512312578E-17 -0.0353498305391302"
+        rpy="0 0 0" />
+      <mass
+        value="0.40765592096642" />
+      <inertia
+        ixx="0.00076152629456158"
+        ixy="2.07681767546495E-05"
+        ixz="-6.15417341469107E-20"
+        iyy="0.000502926266955213"
+        iyz="3.73082590857221E-19"
+        izz="0.000528106575482838" />
     </inertial>
     <visual>
@@ -284,5 +302,5 @@
         name="">
         <color
-          rgba="0.792156862745098 0.819607843137255 0.933333333333333 1" />
+          rgba="0.898039215686275 0.917647058823529 0.929411764705882 1" />
       </material>
     </visual>
@@ -302,5 +320,5 @@
     <origin
       xyz="0 0 0"
-      rpy="-1.5708 0 0.07963" />
+      rpy="0 0 0" />
     <parent
       link="front_wheel_mount_plate_2" />
@@ -308,5 +326,5 @@
       link="front_wheel_holder_2" />
     <axis
-      xyz="0 1 0" />
+      xyz="0 0 -1" />
   </joint>
   <link
@@ -314,15 +332,15 @@
     <inertial>
       <origin
-        xyz="0 0 2.77555756156289E-17"
-        rpy="0 0 0" />
-      <mass
-        value="1.7356" />
-      <inertia
-        ixx="0.0021082"
-        ixy="-3.2526E-19"
-        ixz="1.2945E-18"
-        iyy="0.0021082"
-        iyz="-1.3425E-18"
-        izz="0.0034491" />
+        xyz="5.55111512312578E-17 0 0"
+        rpy="0 0 0" />
+      <mass
+        value="1.73558464244813" />
+      <inertia
+        ixx="0.00211668077407555"
+        ixy="-0.000106327132064745"
+        ixz="-2.97271341358694E-19"
+        iyy="0.00344063904022875"
+        iyz="-1.72056927832268E-21"
+        izz="0.00210819601428248" />
     </inertial>
     <visual>
@@ -337,5 +355,5 @@
         name="">
         <color
-          rgba="0.792156862745098 0.819607843137255 0.933333333333333 1" />
+          rgba="0.898039215686275 0.917647058823529 0.929411764705882 1" />
       </material>
     </visual>
@@ -354,6 +372,6 @@
     type="continuous">
     <origin
-      xyz="0 0.081 0"
-      rpy="0 0 2.2113" />
+      xyz="0 0 -0.081"
+      rpy="0 0 0" />
     <parent
       link="front_wheel_holder_2" />
@@ -361,5 +379,5 @@
       link="front_wheel_2" />
     <axis
-      xyz="0 0 1" />
+      xyz="0.0795457683033873 -0.996831214772603 0" />
   </joint>
   <link
@@ -367,15 +385,15 @@
     <inertial>
       <origin
-        xyz="2.77555756156289E-17 2.77555756156289E-17 0.12370581952403"
-        rpy="0 0 0" />
-      <mass
-        value="3.6906" />
-      <inertia
-        ixx="0.0091266"
-        ixy="5.5702E-19"
-        ixz="-7.4876E-19"
-        iyy="0.010315"
-        iyz="-3.3515E-19"
-        izz="0.0067288" />
+        xyz="-2.77555756156289E-17 0.12370581952403 2.77555756156289E-17"
+        rpy="0 0 0" />
+      <mass
+        value="3.69062219624929" />
+      <inertia
+        ixx="0.00912658772080383"
+        ixy="8.63502453250557E-19"
+        ixz="-5.57023878196132E-19"
+        iyy="0.00672881943632791"
+        iyz="-2.81940192519475E-19"
+        izz="0.0103145877208038" />
     </inertial>
     <visual>
@@ -390,5 +408,5 @@
         name="">
         <color
-          rgba="0.792156862745098 0.819607843137255 0.933333333333333 1" />
+          rgba="0.898039215686275 0.917647058823529 0.929411764705882 1" />
       </material>
     </visual>
@@ -408,5 +426,5 @@
     <origin
       xyz="-0.2185 -0.25 -0.13"
-      rpy="1.5708 0 3.1416" />
+      rpy="0 0 0" />
     <parent
       link="base_link" />
@@ -420,15 +438,15 @@
     <inertial>
       <origin
-        xyz="4.16333634234434E-16 -5.55111512312578E-17 0.0399999999999996"
-        rpy="0 0 0" />
-      <mass
-        value="7.2726" />
-      <inertia
-        ixx="0.025637"
-        ixy="2.647E-22"
-        ixz="2.6866E-18"
-        iyy="0.025637"
-        iyz="-3.1161E-18"
-        izz="0.043516" />
+        xyz="-5.55111512312578E-17 0.0399999999999996 4.16333634234434E-16"
+        rpy="0 0 0" />
+      <mass
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
File: src/trolley_arm_description/urdf/trolley_arm.urdf.xacro (robot description, xacro)
@@ -4,8 +4,8 @@
         <xacro:arg name="ros_namespace" default="toilet_trolley_arm_description"/>
         <!-- load trolley -->
-        <xacro:include filename="$(find hivebot_trolley)/urdf/hivebot_trolley.urdf" />
+        <xacro:include filename="$(find hivebot_trolley)/urdf/hivebot_trolley.xacro" />
         <!-- load mycobot_pro_320 -->
         <xacro:include filename="$(find mycobot_320)/urdf/mycobot_robot_macro.xacro" />
-        <xacro:mycobot_pro_robot_macro attach_to="mount-box" xyz="0 -0.06 -0.06" rpy="0 1.5707 0"/>
+        <xacro:mycobot_pro_robot_macro attach_to="mount-box" xyz="0.05 0 0" rpy="0 1.5707 0"/>
     </xacro:macro>
     <xacro:trolley_arm_macro/>
