Commit message: feat: added toilet_urdf and updated sensors on mycobot

File: src/hivebot_trolley/urdf/hivebot_trolley.xacro (robot description, xacro)
@@ -158,5 +158,5 @@
   <joint
     name="front_wheel_holder_1_toplate"
-    type="continuous">
+    type="fixed">
     <origin
       xyz="0 0 0"
@@ -211,5 +211,5 @@
   <joint
     name="front_wheel_1_toholder"
-    type="continuous">
+    type="fixed">
     <origin
       xyz="0 0 -0.081"
@@ -317,5 +317,5 @@
   <joint
     name="front_wheel_holder_2_toplate"
-    type="continuous">
+    type="fixed">
     <origin
       xyz="0 0 0"
@@ -370,5 +370,5 @@
   <joint
     name="front_wheel_2_toholder"
-    type="continuous">
+    type="fixed">
     <origin
       xyz="0 0 -0.081"
@@ -476,5 +476,5 @@
   <joint
     name="back_wheel_2_toholder"
-    type="continuous">
+    type="fixed">
     <origin
       xyz="0 0 0"
@@ -582,5 +582,5 @@
   <joint
     name="back_wheel_1_toholder"
-    type="continuous">
+    type="fixed">
     <origin
       xyz="0 0 0"
@@ -687,5 +687,5 @@
   </link>
   <joint
-    name="mount-box-to-frame"
+    name="mount_box_to_frame"
     type="prismatic">
     <origin

File: src/mycobot_320/urdf/mycobot_robot.sensor.xacro (robot description, xacro)
@@ -22,5 +22,5 @@
         <visual>
             <geometry>
-                <box size="0.01 0.01 0.01" />
+                <box size="0.02 0.02 0.02" />
             </geometry>
             <material name="Green">
@@ -34,6 +34,6 @@
     </link>
     <joint name="camera_joint" type="fixed">
-        <origin xyz="0 0 0" rpy="0 0 0" />
-        <parent link="j5"/>
+        <origin xyz="0 -0.03 0" rpy="3.14 3.14 0" />
+        <parent link="j6"/>
         <child link="camera_link"/>
     </joint>

File: src/trolley_arm_description/urdf/trolley_arm.urdf.xacro (robot description, xacro)
@@ -3,4 +3,5 @@
     <xacro:macro name="trolley_arm_macro">
         <xacro:arg name="ros_namespace" default="toilet_trolley_arm_description"/>
+        <xacro:arg name="camera_sensor" default="True"/>
         <!-- load trolley -->
         <xacro:include filename="$(find hivebot_trolley)/urdf/hivebot_trolley.xacro" />
@@ -9,5 +10,5 @@
         <!-- include gazebo transmissions -->
         <xacro:include filename="$(find trolley_arm_description)/urdf/trolley_arm.gazebo.xacro"/>
-        <xacro:mycobot_pro_robot_macro attach_to="mount-box" xyz="0.05 0 0" rpy="0 1.5707 0"/>
+        <xacro:mycobot_pro_robot_macro attach_to="mount-box" xyz="0.05 0 0" rpy="0 1.5707 0" camera_sensor="$(arg camera_sensor)"/>
     </xacro:macro>
     <xacro:trolley_arm_macro/>

Commit message: enhancement: updated robot virtual joint tomake it rigidly attached to the world

File: src/hivebot_trolley/urdf/hivebot_trolley.xacro (robot description, xacro)
@@ -4,4 +4,5 @@
      For more information, please see http://wiki.ros.org/sw_urdf_exporter -->
 <robot name="hivebot_trolley">
+  <link name="world"/>
   <link name="base_footprint" xmlns:xacro="http://www.ros.org/wiki/xacro"/>
   <joint name="base_joint" type="fixed">
@@ -1168,3 +1169,8 @@
       xyz="0 0 1" />
   </joint>
+  <joint name="world_base" type="fixed">
+    <origin xyz="0 0 0.2"/>
+    <parent link="world"/>
+    <child link="base_footprint"/>
+  </joint>
 </robot>
